File: t1s_hat/t1s_hat.kicad_sch (KiCad schematic)
At the start: 37 parts, among them CN1 T1S BUS P N N P, J1 2x20 socket (riser stack), U1 LAN8651, Y1 25.000MHz

Commit message: T1S HAT: real choke and varistor lands, both nets closed, silk cleaned
The choke was the fabrication blocker. L1 sat on KiCad's 1206 4-terminal
land (3.2 x 1.6 mm) while every part AN1718 names is 3.2 x 2.5 mm, so the
real component's terminals missed the pads. AN1718 says its part numbers
are examples and the customer picks, so pick one that can be bought:
TDK ACT1210L-201-2P-TL00, 200 uH @ 100 kHz (inside the 130..240 uH span
the three examples cover), AEC-Q200, LCSC C131444. Its land is drawn from
TDK's own ACT1210 layout recommendation -- 4.1 x 1.6 mm overall, 2.0 and
0.4 mm gaps -- into a new project footprint library, and the symbol moves
to L_Coupled_1423 because the ACT1210's windings are 1-4 and 2-3.

MOV1/MOV2 got the same treatment. ELECTRICAL.md already names
TDK AVRH10C221KT1R5YA8, which is a 1005 [0402] part; the board had it on
a 1206 resistor land. Now on a 0402 land taken from TDK's AVR catalogue
recommended pattern. LCSC C2157827. Still DNP.

Both unrouted nets are closed, unrouted count 0, with nothing on B.Cu:

  SPI_CS_N  R5 moved to straddle the MISO column -- MISO passes between
            its own pads. No extra part.
  VDDP      JP1, a real 0 ohm 0603, straddling the +3V3 branch on the
            left edge. In the schematic (net split VDDP / VDDP_17, each
            with its own PWR_FLAG), in the BOM as "fit", and on the silk.

Silkscreen: 48 violations to 0. Designators are now placed by the
generator, which tries each one in a ring around its own part and keeps
the first position clear of every pad, via, ink and the board edge; none
had to be dropped. Board text re-laid into the pad-free areas, CN1's
per-pad letters replaced by a legend, pin-1 marker is a dot.

The all-layer void under the choke is sized to the part: maximum body
3.9 x 2.7 mm plus 0.25 mm a side. It grew in x only because the part did.

Verified: mechanical worst error 0.00000 mm, antenna keepout 0 intruders,
B.Cu signal tracks 0, unrouted 0, ERC 0 errors / 5 warnings, D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
Parts:
- added JP1: 0R jumper, Resistor_SMD:R_0603_1608Metric, symbol Device:R
- L1: value 130uH @ 100kHz CMC -> 200uH @ 100kHz CMC; footprint Inductor_SMD:L_CommonMode_Wurth_WE-CNSW-1206 -> t1s_hat:L_CommonMode_TDK_ACT1210_3225; symbol Device:L_Coupled_1243 -> Device:L_Coupled_1423; LCSC (none) -> C131444
- MOV1, MOV2: value ESD 1206 (DNP) -> 22V 1.5pF ESD (DNP); footprint Resistor_SMD:R_1206_3216Metric -> t1s_hat:Varistor_TDK_AVRH10_1005; LCSC (none) -> C2157827
Connections:
- net CMC_N: now also L1.3; no longer L1.2
- net CMC_P: now also L1.4; no longer L1.3
- net TRXN: now also L1.2; no longer L1.1
- net TRXP: now also L1.1; no longer L1.4
- net VDDP: now also JP1.1; no longer C10.1, C9.1, U1.17 (VDDP)
- new net VDDP_17: C10.1, C9.1, JP1.2, U1.17 (VDDP)
Other:
- note added: "JP1 - 0 ohm link. VDDP is one supply island; on two layers its two halves need one crossing, and JP1 is it. FITTED."
Changed lines of the file:
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@@
     (stroke (width 0) (type default))
   )
-  (label "VDDP" (at 187.96 95.25 90)
+  (label "VDDP_17" (at 187.96 95.25 90)
     (effects (font (size 1.27 1.27)) (justify left bottom))
   )
@@
   )
   (no_connect (at 73.66 154.94))
-  (symbol (lib_id "Device:L_Coupled_1243") (at 275.59 105.41 0) (unit 1)
+  (symbol (lib_id "Device:L_Coupled_1423") (at 275.59 105.41 0) (unit 1)
     (in_bom yes) (on_board yes) (dnp no)
     (property "Reference" "L1" (at 277.79 103.21 0)
       (effects (font (size 1.27 1.27)) (justify left))
     )
-    (property "Value" "130uH @ 100kHz CMC" (at 277.79 106.01 0)
-      (effects (font (size 1.27 1.27)) (justify left))
-    )
-    (property "Footprint" "Inductor_SMD:L_CommonMode_Wurth_WE-CNSW-1206" (at 275.59 105.41 0)
+    (property "Value" "200uH @ 100kHz CMC" (at 277.79 106.01 0)
+      (effects (font (size 1.27 1.27)) (justify left))
+    )
+    (property "Footprint" "t1s_hat:L_CommonMode_TDK_ACT1210_3225" (at 275.59 105.41 0)
       (effects (font (size 1.27 1.27)) hide)
     )
@@
       (effects (font (size 1.27 1.27)) hide)
     )
-    (property "Description" "Common-mode choke, 130 uH @ 100 kHz (AN1718 L1). ALWAYS FITTED." (at 275.59 105.41 0)
+    (property "Description" "Common-mode choke, 2-line, 200 uH @ 100 kHz, EIA 1210 (3.2x2.5 mm), AEC-Q200 - TDK ACT1210L-201-2P-TL00 (AN1718 L1). ALWAYS FITTED." (at 275.59 105.41 0)
+      (effects (font (size 1.27 1.27)) hide)
+    )
+    (property "LCSC" "C131444" (at 275.59 105.41 0)
       (effects (font (size 1.27 1.27)) hide)
     )
@@
     (stroke (width 0) (type default))
   )
-  (label "TRXN" (at 267.97 102.87 0)
-    (effects (font (size 1.27 1.27)) (justify right bottom))
+  (label "TRXP" (at 267.97 102.87 0)
+    (effects (font (size 1.27 1.27)) (justify right bottom))
+  )
+  (wire (pts (xy 270.51 107.95) (xy 267.97 107.95))
+    (stroke (width 0) (type default))
+  )
+  (label "TRXN" (at 267.97 107.95 0)
+    (effects (font (size 1.27 1.27)) (justify right bottom))
+  )
+  (wire (pts (xy 280.67 107.95) (xy 283.21 107.95))
+    (stroke (width 0) (type default))
+  )
+  (label "CMC_N" (at 283.21 107.95 0)
+    (effects (font (size 1.27 1.27)) (justify left bottom))
   )
   (wire (pts (xy 280.67 102.87) (xy 283.21 102.87))
     (stroke (width 0) (type default))
   )
-  (label "CMC_N" (at 283.21 102.87 0)
-    (effects (font (size 1.27 1.27)) (justify left bottom))
-  )
-  (wire (pts (xy 280.67 107.95) (xy 283.21 107.95))
-    (stroke (width 0) (type default))
-  )
-  (label "CMC_P" (at 283.21 107.95 0)
-    (effects (font (size 1.27 1.27)) (justify left bottom))
-  )
-  (wire (pts (xy 270.51 107.95) (xy 267.97 107.95))
-    (stroke (width 0) (type default))
-  )
-  (label "TRXP" (at 267.97 107.95 0)
-    (effects (font (size 1.27 1.27)) (justify right bottom))
+  (label "CMC_P" (at 283.21 102.87 0)
+    (effects (font (size 1.27 1.27)) (justify left bottom))
   )
   (symbol (lib_id "Device:C") (at 299.72 95.25 0) (unit 1)
@@
       (effects (font (size 1.27 1.27)) (justify left))
     )
-    (property "Value" "ESD 1206 (DNP)" (at 387.01 100.93 0)
-      (effects (font (size 1.27 1.27)) (justify left))
-    )
-    (property "Footprint" "Resistor_SMD:R_1206_3216Metric" (at 384.81 100.33 0)
+    (property "Value" "22V 1.5pF ESD (DNP)" (at 387.01 100.93 0)
+      (effects (font (size 1.27 1.27)) (justify left))
+    )
+    (property "Footprint" "t1s_hat:Varistor_TDK_AVRH10_1005" (at 384.81 100.33 0)
       (effects (font (size 1.27 1.27)) hide)
     )
@@
       (effects (font (size 1.27 1.27)) hide)
     )
-    (property "Description" "ESD element on bus P, at the connector (AN1718 MOV1). Optional." (at 384.81 100.33 0)
+    (property "Description" "ESD element on bus P, at the connector (AN1718 MOV1) - TDK AVRH10C221KT1R5YA8 chip varistor, 1005 [0402], 1.5 pF. Optional." (at 384.81 100.33 0)
+      (effects (font (size 1.27 1.27)) hide)
+    )
+    (property "LCSC" "C2157827" (at 384.81 100.33 0)
       (effects (font (size 1.27 1.27)) hide)
     )
@@
       (effects (font (size 1.27 1.27)) (justify left))
     )
-    (property "Value" "ESD 1206 (DNP)" (at 387.01 139.03 0)
-      (effects (font (size 1.27 1.27)) (justify left))
-    )
-    (property "Footprint" "Resistor_SMD:R_1206_3216Metric" (at 384.81 138.43 0)
+    (property "Value" "22V 1.5pF ESD (DNP)" (at 387.01 139.03 0)
+      (effects (font (size 1.27 1.27)) (justify left))
+    )
+    (property "Footprint" "t1s_hat:Varistor_TDK_AVRH10_1005" (at 384.81 138.43 0)
       (effects (font (size 1.27 1.27)) hide)
     )
@@
       (effects (font (size 1.27 1.27)) hide)
     )
-    (property "Description" "ESD element on bus N, at the connector (AN1718 MOV2). Optional." (at 384.81 138.43 0)
+    (property "Description" "ESD element on bus N, at the connector (AN1718 MOV2) - TDK AVRH10C221KT1R5YA8 chip varistor, 1005 [0402], 1.5 pF. Optional." (at 384.81 138.43 0)
+      (effects (font (size 1.27 1.27)) hide)
+    )
+    (property "LCSC" "C2157827" (at 384.81 138.43 0)
       (effects (font (size 1.27 1.27)) hide)
     )
@@
     (stroke (width 0) (type default))
   )
-  (label "VDDP" (at 115.57 38.10 90)
+  (label "VDDP_17" (at 115.57 38.10 90)
     (effects (font (size 1.27 1.27)) (justify left bottom))
   )
@@
     (stroke (width 0) (type default))
   )
-  (label "VDDP" (at 130.81 38.10 90)
+  (label "VDDP_17" (at 130.81 38.10 90)
     (effects (font (size 1.27 1.27)) (justify left bottom))
   )
@@
       (effects (font (size 1.27 1.27)) hide)
     )
-    (property "Description" "SPI CS_N pull-up" (at 110.49 124.46 0)
+    (property "Description" "SPI CS_N pull-up; also the F.Cu crossover for SPI_MISO, which passes between its pads" (at 110.49 124.46 0)
       (effects (font (size 1.27 1.27)) hide)
     )
@@
     (effects (font (size 1.27 1.27)) (justify left bottom))
   )
+  (symbol (lib_id "Device:R") (at 110.49 80.01 0) (unit 1)
+    (in_bom yes) (on_board yes) (dnp no)
+    (property "Reference" "JP1" (at 112.69 77.81 0)
+      (effects (font (size 1.27 1.27)) (justify left))
+    )
+    (property "Value" "0R jumper" (at 112.69 80.61 0)
+      (effects (font (size 1.27 1.27)) (justify left))
+    )
+    (property "Footprint" "Resistor_SMD:R_0603_1608Metric" (at 110.49 80.01 0)
+      (effects (font (size 1.27 1.27)) hide)
+    )
+    (property "Datasheet" "" (at 110.49 80.01 0)
+      (effects (font (size 1.27 1.27)) hide)
+    )
+    (property "Description" "0 ohm link, VDDP pin-7 island to VDDP pin-17 island. The 2-layer crossover for +3V3, which passes between its pads. FITTED - the board does not work without it." (at 110.49 80.01 0)
+      (effects (font (size 1.27 1.27)) hide)
+    )
+    (pin "1")
+    (pin "2")
+    (instances (project "t1s_hat" (path "/5f3b7c10-1a2b-4c3d-8e9f-0a1b2c3d4e50"
+      (reference "JP1") (unit 1)
+    )))
+  )
+  (wire (pts (xy 110.49 76.20) (xy 110.49 73.66))
+    (stroke (width 0) (type default))
+  )
+  (label "VDDP" (at 110.49 73.66 90)
+    (effects (font (size 1.27 1.27)) (justify left bottom))
+  )
+  (wire (pts (xy 110.49 83.82) (xy 110.49 86.36))
+    (stroke (width 0) (type default))
+  )
+  (label "VDDP_17" (at 110.49 86.36 270)
+    (effects (font (size 1.27 1.27)) (justify right bottom))
+  )
   (symbol (lib_id "power:PWR_FLAG") (at 39.37 250.19 0) (unit 1)
     (in_bom no) (on_board yes) (dnp no)
@@
     (stroke (width 0) (type default))
   )
-  (label "VDDA" (at 135.89 250.19 0)
+  (label "VDDP_17" (at 135.89 250.19 0)
     (effects (font (size 1.27 1.27)) (justify left bottom))
   )
@@
     (stroke (width 0) (type default))
   )
-  (label "VDDAU" (at 166.37 250.19 0)
+  (label "VDDA" (at 166.37 250.19 0)
+    (effects (font (size 1.27 1.27)) (justify left bottom))
+  )
+  (symbol (lib_id "power:PWR_FLAG") (at 191.77 250.19 0) (unit 1)
+    (in_bom no) (on_board yes) (dnp no)
+    (property "Reference" "#FLG055" (at 193.97 247.99 0)
+      (effects (font (size 1.27 1.27)) (justify left) hide)
+    )
+    (property "Value" "PWR_FLAG" (at 193.97 250.79 0)
+      (effects (font (size 1.27 1.27)) (justify left) hide)
+    )
+    (property "Datasheet" "" (at 191.77 250.19 0)
+      (effects (font (size 1.27 1.27)) hide)
+    )
+    (pin "1")
+    (instances (project "t1s_hat" (path "/5f3b7c10-1a2b-4c3d-8e9f-0a1b2c3d4e50"
+      (reference "#FLG055") (unit 1)
+    )))
+  )
+  (wire (pts (xy 191.77 250.19) (xy 196.85 250.19))
+    (stroke (width 0) (type default))
+  )
+  (label "VDDAU" (at 196.85 250.19 0)
     (effects (font (size 1.27 1.27)) (justify left bottom))
   )
@@
     (effects (font (size 1.80 1.80) bold) (justify left bottom))
   )
+  (text "JP1 - 0 ohm link. VDDP is one supply island; on two layers its two halves need one crossing, and JP1 is it. FITTED." (at 60.00 76.00 0)
+    (effects (font (size 1.80 1.80) bold) (justify left bottom))
+  )
